File: clock61/clock61.kicad_pcb (KiCad board)
At the start: 2 copper layers, 55.2 x 55.2 mm, 78 parts

Commit message: wip
Parts:
- removed 0, 2, 3, 4, 5, 6, 7: 1, min:hand
- removed 0, 1, 3, 4, 5, 6, 7: 2, min:hand
- removed 0, 1, 2, 4, 5, 6, 7: 3, min:hand
- removed 0, 1, 2, 3, 5, 6: 4, min:hand
- removed 0, 1, 2, 3, 4, 6: 5, min:hand
- removed 0, 1, 2, 3, 4, 5: 6, min:hand
- removed 0, 1, 2, 3, 4, 5, 6: 7, min:hand
- removed 0, 1, 2, 3, 4, 5, 6: 8, min:hand
- removed 1, 2, 3, 4, 5, 6, 7: 0, min:hand
- removed x (x9): x, resi:stor
- removed x (x9): x, pin:hole
- added ? (x60): , min:hand, F.Cu at (150.0, 100.0)
- added ? (x9): , resi:stor, F.Cu at (150.0, 100.0)
- added ?: , pin:hole, F.Cu at (156.0, 93.3)
- added ?: , pin:hole, F.Cu at (149.1, 91.0)
- added ?: , pin:hole, F.Cu at (159.0, 100.0)
- added ?: , pin:hole, F.Cu at (142.7, 94.7)
- added ?: , pin:hole, F.Cu at (141.2, 101.9)
- added ?: , pin:hole, F.Cu at (145.5, 107.8)
- added ?: , pin:hole, F.Cu at (152.8, 108.6)
- added ?: , pin:hole, F.Cu at (158.2, 103.7)
- added ?: , pin:hole, F.Cu at (150.0, 100.0)

Commit message: wip
Parts:
- removed the ? at (150.0, 100.0) (x69)
- added ? (x60): , min:hand, F.Cu at (150.0, 100.0)
- added ? (x9): , resi:stor, F.Cu at (150.0, 100.0)
- added x: x, mounting:hole, F.Cu at (125.4, 75.4)
- added x: x, mounting:hole, F.Cu at (125.4, 124.6)
- added x: x, mounting:hole, F.Cu at (174.6, 75.4)
- added x: x, mounting:hole, F.Cu at (174.6, 124.6)
Other:
- board text added: "clock61"
Changed lines of the file:
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@@
   (gr_line (start    122.400     72.400 ) (end     177.600      72.400 ) (angle  0) (layer Edge.Cuts) (width 0.15))
   (gr_line (start    122.400    127.600 ) (end     177.600     127.600 ) (angle  0) (layer Edge.Cuts) (width 0.15))
+  (module mounting:hole (layer F.Cu)
+    (at 125.400 75.400)
+    (descr hole)
+    (tags hole)
+    (fp_text reference x (at 0 0) (layer F.Fab) (effects (font (size 1 1) (thickness 0.15))))
+    (fp_text value     x (at 0 0) (layer F.Fab) (effects (font (size 1 1) (thickness 0.15))))
+    (pad 1 thru_hole circle (at 0 0) (size 3 3) (drill 3) (layers *.Cu *.Mask F.SilkS))
+  )
+  (module mounting:hole (layer F.Cu)
+    (at 125.400 124.600)
+    (descr hole)
+    (tags hole)
+    (fp_text reference x (at 0 0) (layer F.Fab) (effects (font (size 1 1) (thickness 0.15))))
+    (fp_text value     x (at 0 0) (layer F.Fab) (effects (font (size 1 1) (thickness 0.15))))
+    (pad 1 thru_hole circle (at 0 0) (size 3 3) (drill 3) (layers *.Cu *.Mask F.SilkS))
+  )
+  (module mounting:hole (layer F.Cu)
+    (at 174.600 75.400)
+    (descr hole)
+    (tags hole)
+    (fp_text reference x (at 0 0) (layer F.Fab) (effects (font (size 1 1) (thickness 0.15))))
+    (fp_text value     x (at 0 0) (layer F.Fab) (effects (font (size 1 1) (thickness 0.15))))
+    (pad 1 thru_hole circle (at 0 0) (size 3 3) (drill 3) (layers *.Cu *.Mask F.SilkS))
+  )
+  (module mounting:hole (layer F.Cu)
+    (at 174.600 124.600)
+    (descr hole)
+    (tags hole)
+    (fp_text reference x (at 0 0) (layer F.Fab) (effects (font (size 1 1) (thickness 0.15))))
+    (fp_text value     x (at 0 0) (layer F.Fab) (effects (font (size 1 1) (thickness 0.15))))
+    (pad 1 thru_hole circle (at 0 0) (size 3 3) (drill 3) (layers *.Cu *.Mask F.SilkS))
+  )
+(gr_text clock61 (at 150  97) (layer B.Cu) (effects (font (size 1.5 1.5) (thickness 0.3))(justify mirror)) )
 )
