File: clock61/version3/clock61.kv3.kicad_pcb (KiCad board)
At the start: 2 copper layers, 55.2 x 55.2 mm, 82 parts

Commit message: subtle changes to make a kicad version 3 file so more folks can view it
Parts:
- removed the ? at (150.0, 100.0) (x69)
- added ? (x60): , min:hand, F.Cu at (150.0, 100.0)
- added ? (x9): , resi:stor, F.Cu at (150.0, 100.0)
Other:
- net class Default: clearance 0.2 -> 0.254; trace_width 0.25 -> 0.254; via_dia 0.6 -> 0.889; via_drill 0.4 -> 0.635
- rule trace_clearance: 0.2 -> 0.254
- rule trace_min: 0.2 -> 0.254
- rule via_min_drill: 0.3 -> 0.508
- rule via_min_size: 0.4 -> 0.889
