File: clock7/clock7a.kicad_pcb (KiCad board)
At the start: 2 copper layers, 12 parts

Commit message: wip
Parts:
- added ?: , my_modules:STM32_LQFP32, B.Cu at (74.4, 82.5)
Routing:
- net (no net): track 727.1 -> 918.9 mm, vias 31 -> 34

Commit message: wip
Parts:
- added ?: , 00my_modules:gps, F.Cu at (111.7, 72.3)
- added ?: , 00my_modules:UE27-BC54-130, B.Cu at (58.7, 82.5)
- added ?: , 00my_modules:AP2112, B.Cu at (68.1, 76.7)
- added ?: C, 00my_modules:R_0603, B.Cu at (63.2, 75.4)
- added ?: C, 00my_modules:R_0603, B.Cu at (63.2, 73.9)
- added ?: R, 00my_modules:R_0603, B.Cu at (79.8, 93.0)
- added ?: , 00my_modules:Pin_Header_Straight_1x04, F.Cu at (71.6, 70.9)
- added ?: R, 00my_modules:R_0603, B.Cu at (79.8, 75.2)
- added ?: , 00my_modules:Hole0, F.Cu at (147.3, 70.4)
- added ?: , 00my_modules:Hole0, F.Cu at (147.3, 97.8)
- added ?: , 00my_modules:Hole0, F.Cu at (53.1, 70.4)
- added ?: , 00my_modules:Hole0, F.Cu at (53.1, 97.8)
- added BOOT0: , 00my_modules:BUTTON4, B.Cu at (85.9, 72.9)
- added RESET: , 00my_modules:BUTTON4, B.Cu at (85.9, 95.2)
Routing:
- net (no net): track 918.9 -> 1203.3 mm, vias 34 -> 41
Other:
- board outline added: 103.4 x 36.6 mm
- board text added: "C"
- board text added: "D"
- board text added: "G"
- board text added: "V"
