File: clock7/clock7a_breakout_tabs.kicad_pcb (KiCad board)
At the start: 2 copper layers, 59.2 x 18.8 mm, 12 parts

Commit message: wip
Parts:
- removed the ? at (89.2, 90.2)
- removed the ? at (86.4, 89.2)
- removed the ? at (89.2, 88.1)
- removed the ? at (86.4, 87.1)
- removed the ? at (89.2, 86.1)
- removed the ? at (86.4, 85.1)
- removed the ? at (89.2, 84.1)
- removed the ? at (86.4, 83.1)
- added ?: R, 00my_modules:R_0603, B.Cu at (88.9, 75.2)
- added ?: R, 00my_modules:R_0603, B.Cu at (88.9, 77.7)
- added ?: , 00my_modules:Hole0, F.Cu at (151.1, 84.1)
- added ?: , 00my_modules:Hole0, F.Cu at (79.8, 84.1)
- added ?: , 00my_modules:Pin_Header_Straight_1x08, F.Cu at (85.6, 75.2)
- added ?: , 00my_modules:Pin_Header_Straight_1x04, F.Cu at (145.3, 80.3)
- added ?: R, 00my_modules:R_0603, B.Cu at (88.9, 93.0)
- added ?: R, 00my_modules:R_0603, B.Cu at (88.9, 90.4)
- added ?: R, 00my_modules:R_0603, B.Cu at (88.9, 87.9)
- added ?: R, 00my_modules:R_0603, B.Cu at (88.9, 85.3)
- added ?: R, 00my_modules:R_0603, B.Cu at (88.9, 82.8)
- added ?: R, 00my_modules:R_0603, B.Cu at (88.9, 80.3)
Routing:
- net (no net): track 727.1 -> 713.0 mm
Other:
- board size 59.2 x 18.8 mm -> 79.5 x 21.3 mm
- board text added: "clock7_breakout_tabs"
