File: stuff/gpsxbee.kicad_pcb (KiCad board)
At the start: 2 copper layers, 25.4 x 42.3 mm, 14 parts

Commit message: wip
Routing:
- net (no net): track 190.8 -> 163.1 mm
- net /gnd: track 43.4 -> 71.1 mm
Other:
- board text added: "messed up here, these two are not spaced the same should be closer to - and v"
Changed lines of the file:
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@@
 (kicad_pcb (version 4) (host pcbnew 4.0.7-e2-6376~58~ubuntu16.04.1)
   (general
-    (links 0)
-    (no_connects 0)
+    (links 2)
+    (no_connects 1)
     (area 97.794999 82.394999 128.205001 148.605001)
     (thickness 1.6)
-    (drawings 20)
+    (drawings 25)
     (tracks 66)
     (zones 0)
@@
     (pad - thru_hole circle (at -1.25 -2.7) (size 1.5 1.5) (drill 0.92) (layers *.Cu *.Mask F.SilkS))
     (pad + thru_hole circle (at -1.25 0.5) (size 1.5 1.5) (drill 0.92) (layers *.Cu *.Mask F.SilkS))
-    (pad G thru_hole circle (at 1.25 0.5) (size 1.5 1.5) (drill 0.92) (layers *.Cu *.Mask F.SilkS) (net 1 /gnd) )
+    (pad G thru_hole circle (at 1.25 0.5) (size 1.5 1.5) (drill 0.92) (layers *.Cu *.Mask F.SilkS)
+      (net 1 /gnd))
     (pad X thru_hole circle (at 6.02 0) (size 3.5 3.5) (drill 2.3) (layers *.Cu *.Mask F.SilkS))
     (pad X thru_hole circle (at -6.02 0) (size 3.5 3.5) (drill 2.3) (layers *.Cu *.Mask F.SilkS))
@@
     (pad - thru_hole circle (at -1.25 2.7) (size 1.5 1.5) (drill 0.92) (layers *.Cu *.Mask B.SilkS))
     (pad + thru_hole circle (at -1.25 -0.5) (size 1.5 1.5) (drill 0.92) (layers *.Cu *.Mask B.SilkS))
-    (pad G thru_hole circle (at 1.25 -0.5) (size 1.5 1.5) (drill 0.92) (layers *.Cu *.Mask B.SilkS)(net 1 /gnd) )
+    (pad G thru_hole circle (at 1.25 -0.5) (size 1.5 1.5) (drill 0.92) (layers *.Cu *.Mask B.SilkS)
+      (net 1 /gnd))
     (pad X thru_hole circle (at 6.02 0) (size 3.5 3.5) (drill 2.3) (layers *.Cu *.Mask B.SilkS))
     (pad X thru_hole circle (at -6.02 0) (size 3.5 3.5) (drill 2.3) (layers *.Cu *.Mask B.SilkS))
@@
     (pad 3 thru_hole oval (at 0 2.54 90) (size 2.032 1.7272) (drill 1.016) (layers *.Cu *.Mask F.SilkS))
   )
+  (gr_text "messed up here, these two are not spaced the same should be closer to - and v\n" (at 134.8 113.65) (layer F.Fab)
+    (effects (font (size 1.5 1.5) (thickness 0.3)))
+  )
+  (gr_line (start 134.55 111.45) (end 134.5 111.5) (angle 90) (layer F.Fab) (width 0.2))
+  (gr_line (start 130.3 111.45) (end 134.55 111.45) (angle 90) (layer F.Fab) (width 0.2))
+  (gr_line (start 114.25 127.5) (end 130.3 111.45) (angle 90) (layer F.Fab) (width 0.2))
+  (gr_line (start 114.2 127.5) (end 114.35 127.5) (angle 90) (layer Cmts.User) (width 0.2))
   (gr_text gpsxbee (at 113 136.5) (layer B.SilkS)
     (effects (font (size 1.5 1.5) (thickness 0.3)) (justify mirror))
@@
   (segment (start 103.69 124.74) (end 103.69 99.29) (width 0.25) (layer B.Cu) (net 0))
   (segment (start 103.69 124.74) (end 101.65 126.78) (width 0.25) (layer B.Cu) (net 0))
-  (segment (start 122.85 131) (end 116.14 131) (width 0.25) (layer F.Cu) (net 0))
   (segment (start 124.35 129.2) (end 124.35 127.675) (width 0.25) (layer F.Cu) (net 0))
   (segment (start 121.75 130.275) (end 114.675 130.275) (width 0.25) (layer B.Cu) (net 0))
@@
   (segment (start 101.65 126.78) (end 101.65 125.3) (width 0.25) (layer F.Cu) (net 0))
   (segment (start 101.65 125.3) (end 101.8 125.15) (width 0.25) (layer F.Cu) (net 0))
-  (segment (start 114.25 133.9) (end 114.25 133.875) (width 0.25) (layer F.Cu) (net 0))
-  (segment (start 114.25 133.875) (end 112.675 132.3) (width 0.25) (layer F.Cu) (net 0))
-  (segment (start 108.9 131) (end 103.15 131) (width 0.25) (layer F.Cu) (net 0))
-  (segment (start 110.2 132.3) (end 108.9 131) (width 0.25) (layer F.Cu) (net 0))
-  (segment (start 112.675 132.3) (end 110.2 132.3) (width 0.25) (layer F.Cu) (net 0))
   (segment (start 101.65 129.2) (end 101.65 132.8) (width 0.25) (layer F.Cu) (net 0))
   (segment (start 101.65 129.2) (end 101.65 132.8) (width 0.25) (layer F.Cu) (net 0))
-  (segment (start 113.75 127) (end 114.25 127.5) (width 0.25) (layer F.Cu) (net 0))
   (segment (start 104.6 125.15) (end 105.32 125.15) (width 0.25) (layer F.Cu) (net 0))
   (segment (start 105.32 125.15) (end 106.265 124.205) (width 0.25) (layer F.Cu) (net 0))
@@
   (segment (start 110.56 128.98) (end 109.88 128.3) (width 0.25) (layer F.Cu) (net 0))
   (segment (start 112.53 128.98) (end 110.56 128.98) (width 0.25) (layer F.Cu) (net 0))
-  (segment (start 114.25 133.9) (end 114.25 133.89) (width 0.25) (layer F.Cu) (net 0))
-  (segment (start 114.25 127.5) (end 116.14 129.39) (width 0.25) (layer F.Cu) (net 0))
-  (segment (start 116.14 132.01) (end 114.25 133.9) (width 0.25) (layer F.Cu) (net 0))
-  (segment (start 116.14 129.39) (end 116.14 131) (width 0.25) (layer F.Cu) (net 0))
-  (segment (start 116.14 131) (end 116.14 132.01) (width 0.25) (layer F.Cu) (net 0))
+  (segment (start 122.85 131) (end 116.14 131) (width 0.25) (layer F.Cu) (net 1))
+  (segment (start 114.25 133.9) (end 114.25 133.875) (width 0.25) (layer F.Cu) (net 1))
+  (segment (start 114.25 133.875) (end 112.675 132.3) (width 0.25) (layer F.Cu) (net 1))
+  (segment (start 108.9 131) (end 103.15 131) (width 0.25) (layer F.Cu) (net 1))
+  (segment (start 110.2 132.3) (end 108.9 131) (width 0.25) (layer F.Cu) (net 1))
+  (segment (start 112.675 132.3) (end 110.2 132.3) (width 0.25) (layer F.Cu) (net 1))
+  (segment (start 113.75 127) (end 114.25 127.5) (width 0.25) (layer F.Cu) (net 1))
+  (segment (start 114.25 133.9) (end 114.25 133.89) (width 0.25) (layer F.Cu) (net 1))
+  (segment (start 114.25 127.5) (end 116.14 129.39) (width 0.25) (layer F.Cu) (net 1))
+  (segment (start 116.14 132.01) (end 114.25 133.9) (width 0.25) (layer F.Cu) (net 1))
+  (segment (start 116.14 129.39) (end 116.14 131) (width 0.25) (layer F.Cu) (net 1))
+  (segment (start 116.14 131) (end 116.14 132.01) (width 0.25) (layer F.Cu) (net 1))
   (segment (start 109.25 108.43) (end 109.25 98) (width 0.25) (layer B.Cu) (net 1))
   (segment (start 106.71 110.92) (end 109.25 108.43) (width 0.25) (layer B.Cu) (net 1))
